File: gachi_Master/gachi_Master.kicad_sch (KiCad schematic)
At the start: 19 parts, among them X1 USB_C_Receptacle_USB2.0_16P

Commit message: Add files via upload
Parts:
- added R9: 10k, Resistor_SMD:R_0603_1608Metric, symbol Device:R
- added SW1: SW_Push, symbol Switch:SW_Push
- added VD2, VD3, VD4, VD5: LED, LED_SMD:LED_0603_1608Metric, symbol Device:LED
Connections:
- net GND: now also SW1.2
- net at DD1.2 (LED1): now also VD2.2 (A), VD4.1 (K)
- net at DD1.3 (LED2): now also VD3.2 (A), VD5.1 (K)
- net at DD1.4 (LED3): now also VD2.1 (K), VD3.1 (K), VD4.2 (A), VD5.2 (A)
- net at DD1.5 (KEY): now also R9.2
- net +3.3V renamed 3,3 В
- net +5V renamed 5 В
- new net: R9.1, SW1.1
- no-connect marks 13 -> 9
Other:
- moved on the sheet: BT1, C1, C2, C3, C4, L1, R1, R2, X1
