File: gachi_Master/gachi_master_(stm32&co).kicad_sch (KiCad schematic)
At the start: 26 parts, among them U1 STM32F407VGTx, X2 Conn_01x04

Commit message: Add files via upload
Parts:
- removed R5: 300, Resistor_SMD:R_0603_1608Metric, symbol Device:R
- added C29, C30: 18пФ, Capacitor_SMD:C_0603_1608Metric, symbol Device:C
- added SW2: SW_Push, symbol Switch:SW_Push
- added ZQ1: WTL5M85611FO, Crystal:Crystal_SMD_WE_IQXC-42-4Pin_2.0x1.6mm, symbol Device:Crystal
- VD1: footprint LED_SMD:LED_0201_0603Metric -> LED_SMD:LED_0603_1608Metric
- renumbered U1 to DD3
Connections:
- net GND: now also C29.2, C30.2, SW2.2
- net RS485_RTS: now also DD3.95 (PB8); no longer R7.2
- net RS485_TX: now also DD3.92 (PB6)
- net at C20.2, DD3.14 (NRST), R3.2: now also SW2.1
- net at R7.1: now also DD3.25 (PA2); no longer DD3.95 (PB8)
- net OSC_IN: now reaches DD3.12 (PH0)
- net OSC_IN: now also C30.1, ZQ1.2
- net OSC_OUT: now reaches DD3.13 (PH1)
- net OSC_OUT: now also C29.1, ZQ1.1
- net DWIN_TX: now reaches DD3.24 (PA1)
- new net DWIN_RX: R7.2
Other:
- moved on the sheet: C20, C21, C22, C27, R3, R4

Commit message: update_10.10.2026
Parts:
- added C31: 10пФ, Capacitor_SMD:C_0603_1608Metric, symbol Device:C
- added C32: 10Ф, Capacitor_SMD:C_0603_1608Metric, symbol Device:C
- added ZQ2: 32.768, symbol Device:Crystal
Connections:
- net DWIN_TX: now also DD3.23 (PA0); no longer DD3.24 (PA1)
- net GND: now also C31.2, C32.2
- net RS485_RTS: now also DD3.67 (PA8); no longer DD3.95 (PB8)
- net RS485_TX: now also DD3.68 (PA9); no longer DD3.92 (PB6)
- net at R7.1: now also DD3.24 (PA1); no longer DD3.25 (PA2)
- net at R6.1: now also DD3.69 (PA10); no longer DD3.93 (PB7)
- net ESP_RX: now reaches DD3.26 (PA3)
- net OSC_IN_LSE: now reaches DD3.8 (PC14)
- net OSC_IN_LSE: now also C31.1, ZQ2.2
- net OSC_OUT_LSE: now reaches DD3.9 (PC15)
- net OSC_OUT_LSE: now also C32.1, ZQ2.1
- net OSC_IN renamed OSC_IN_HSE
- net OSC_OUT renamed OSC_OUT_HSE
- new net ESP_TX: DD3.25 (PA2)
Other:
- moved on the sheet: C27, C29, C30, R4, R6, R7, ZQ1

Commit message: update_10.10.2026_2
Parts:
- removed R6: 300, Resistor_SMD:R_0603_1608Metric, symbol Device:R
Connections:
- net RS485_RX: now also DD3.69 (PA10)
Changed lines of the file:
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@@
 	(wire
 		(pts
-			(xy 237.49 111.76) (xy 307.34 111.76)
+			(xy 237.49 111.76) (xy 314.96 111.76)
 		)
 		(stroke
@@
 					(unit 1)
 				)
-			)
-		)
-	)
-	(symbol
-		(lib_id "Device:R")
-		(at 311.15 111.76 90)
-		(unit 1)
-		(body_style 1)
-		(exclude_from_sim no)
-		(in_bom yes)
-		(on_board yes)
-		(in_pos_files yes)
-		(dnp no)
-		(property "Reference" "R6"
-			(at 311.15 106.426 90)
-			(show_name no)
-			(do_not_autoplace no)
-			(effects
-				(font
-					(size 1.27 1.27)
-				)
-			)
-		)
-		(property "Value" "300"
-			(at 311.15 108.966 90)
-			(show_name no)
-			(do_not_autoplace no)
-			(effects
-				(font
-					(size 1.27 1.27)
-				)
-			)
-		)
-		(property "Footprint" "Resistor_SMD:R_0603_1608Metric"
-			(at 311.15 113.538 90)
-			(hide yes)
-			(show_name no)
-			(do_not_autoplace no)
-			(effects
-				(font
-					(size 1.27 1.27)
-				)
-			)
-		)
-		(property "Datasheet" ""
-			(at 311.15 111.76 0)
-			(hide yes)
-			(show_name no)
-			(do_not_autoplace no)
-			(effects
-				(font
-					(size 1.27 1.27)
-				)
-			)
-		)
-		(property "Description" "Resistor"
-			(at 311.15 111.76 0)
-			(hide yes)
-			(show_name no)
-			(do_not_autoplace no)
-			(effects
-				(font
-					(size 1.27 1.27)
-				)
-			)
-		)
-		(pin "1"
-		)
-		(pin "2"
-		)
-		(instances
-			(project "gachi_Master"
-				(path "/ab3207bc-bcd8-4d0f-899e-74aada9f2221"
-					(reference "R6")
-					(unit 1)
-				)
