File: gachi_Master/gachi_master_(rs-485).kicad_sch (KiCad schematic)
At the start: 9 parts, among them X4 Conn_01x02_Pin

Commit message: update_10.10.2026_AF_4
Parts:
- R11: value 300 -> 120
Changed lines of the file:
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@@
 			)
 		)
-		(property "Value" "300"
+		(property "Value" "120"
 			(at 235.712 145.034 0)
 			(show_name no)
